File: tps61040.sch (EAGLE design)
At the start: 10 parts, among them U1 TPS61040DBVR

Commit message: switch to 0603 sized components
Parts:
- C_FF, C_IN, C_O: device Passive_Capacitors_rev15a:WCAP-CSGP_0805-WAVE -> Passive_Capacitors_rev15a:WCAP-CSGP_0603-REFLOW
- R2: device rcl:R-EU_R0805 -> rcl:R-EU_R0603
Changed lines of the file:
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@@
 <setting verticaltext="up"/>
 </settings>
-<grid distance="1.27" unitdist="mm" unit="mm" style="lines" multiple="1" display="no" altdistance="0.127" altunitdist="mm" altunit="mm"/>
+<grid distance="0.1" unitdist="inch" unit="inch" style="lines" multiple="1" display="no" altdistance="0.01" altunitdist="inch" altunit="inch"/>
 <layers>
 <layer number="1" name="Top" color="4" fill="1" visible="no" active="no"/>
@@
 <parts>
 <part name="U1" library="TPS61040DBVR" deviceset="TPS61040DBVR" device=""/>
-<part name="C_IN" library="Passive_Capacitors_rev15a" deviceset="WCAP-CSGP" device="_0805-WAVE" value="4.7uF"/>
-<part name="C_FF" library="Passive_Capacitors_rev15a" deviceset="WCAP-CSGP" device="_0805-WAVE" value="22pF"/>
-<part name="C_O" library="Passive_Capacitors_rev15a" deviceset="WCAP-CSGP" device="_0805-WAVE" value="1uF"/>
+<part name="C_IN" library="Passive_Capacitors_rev15a" deviceset="WCAP-CSGP" device="_0603-REFLOW" value="4.7uF"/>
+<part name="C_FF" library="Passive_Capacitors_rev15a" deviceset="WCAP-CSGP" device="_0603-REFLOW" value="22pF"/>
+<part name="C_O" library="Passive_Capacitors_rev15a" deviceset="WCAP-CSGP" device="_0603-REFLOW" value="1uF"/>
 <part name="SV1" library="con-lstb" library_urn="urn:adsk.eagle:library:162" deviceset="MA04-1" device="" package3d_urn="urn:adsk.eagle:package:8337/1"/>
 <part name="EN_J" library="jumper" library_urn="urn:adsk.eagle:library:252" deviceset="SJ" device="" package3d_urn="urn:adsk.eagle:package:15471/1"/>
@@
 <part name="D1" library="SS54" deviceset="SS54" device=""/>
 <part name="VR1" library="TC33X-2-103G" deviceset="TC33X-2-103G" device="" value="10k"/>
-<part name="R2" library="rcl" library_urn="urn:adsk.eagle:library:334" deviceset="R-EU_" device="R0805" package3d_urn="urn:adsk.eagle:package:23553/2" value="1k"/>
+<part name="R2" library="rcl" library_urn="urn:adsk.eagle:library:334" deviceset="R-EU_" device="R0603" package3d_urn="urn:adsk.eagle:package:23555/3" value="1k"/>
 </parts>
 <sheets>

Commit message: update schematics to v1.1
Parts:
- removed SV1: (no value), con-lstb:MA04-1
- added EN, GND, VIN, VOUT: TPB1,27, testpad:TPB1,27
- added R1: Xk, rcl:R-EU_R0603
Connections:
- net EN: now also EN.TP; no longer SV1.4
- net GND: now also GND.TP; no longer SV1.1
- net N$2: now also R1.1
- net VIN: now also VIN.TP; no longer SV1.3
- net VOUT: now also R1.2, VOUT.TP; no longer SV1.2
Changed lines of the file:
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@@
 <part name="C_FF" library="Passive_Capacitors_rev15a" deviceset="WCAP-CSGP" device="_0603-REFLOW" value="22pF"/>
 <part name="C_O" library="Passive_Capacitors_rev15a" deviceset="WCAP-CSGP" device="_0603-REFLOW" value="1uF"/>
-<part name="SV1" library="con-lstb" library_urn="urn:adsk.eagle:library:162" deviceset="MA04-1" device="" package3d_urn="urn:adsk.eagle:package:8337/1"/>
 <part name="EN_J" library="jumper" library_urn="urn:adsk.eagle:library:252" deviceset="SJ" device="" package3d_urn="urn:adsk.eagle:package:15471/1"/>
 <part name="L1" library="cd43" library_urn="urn:adsk.eagle:library:44842319" deviceset="CD43" device="" package3d_urn="urn:adsk.eagle:package:44842322/2" value="10uH"/>
@@
 <part name="VR1" library="TC33X-2-103G" deviceset="TC33X-2-103G" device="" value="10k"/>
 <part name="R2" library="rcl" library_urn="urn:adsk.eagle:library:334" deviceset="R-EU_" device="R0603" package3d_urn="urn:adsk.eagle:package:23555/3" value="1k"/>
+<part name="R1" library="rcl" library_urn="urn:adsk.eagle:library:334" deviceset="R-EU_" device="R0603" package3d_urn="urn:adsk.eagle:package:23555/3" value="Xk"/>
+<part name="GND" library="testpad" library_urn="urn:adsk.eagle:library:385" deviceset="TP" device="B1,27" package3d_urn="urn:adsk.eagle:package:27944/2"/>
+<part name="VOUT" library="testpad" library_urn="urn:adsk.eagle:library:385" deviceset="TP" device="B1,27" package3d_urn="urn:adsk.eagle:package:27944/2"/>
+<part name="VIN" library="testpad" library_urn="urn:adsk.eagle:library:385" deviceset="TP" device="B1,27" package3d_urn="urn:adsk.eagle:package:27944/2"/>
+<part name="EN" library="testpad" library_urn="urn:adsk.eagle:library:385" deviceset="TP" device="B1,27" package3d_urn="urn:adsk.eagle:package:27944/2"/>
 </parts>
 <sheets>
@@
 <attribute name="VALUE" x="110.744" y="58.801" size="1.27" layer="96"/>
 </instance>
-<instance part="SV1" gate="1" x="7.62" y="48.26" smashed="yes">
-<attribute name="VALUE" x="6.35" y="40.64" size="1.778" layer="96"/>
-<attribute name="NAME" x="6.35" y="54.102" size="1.27" layer="95"/>
-</instance>
 <instance part="EN_J" gate="1" x="25.4" y="73.66" smashed="yes" rot="R90">
 <attribute name="NAME" x="22.86" y="71.12" size="1.27" layer="95" rot="R90"/>
@@
 <attribute name="NAME" x="86.1314" y="50.8" size="1.27" layer="95" rot="R90"/>
 <attribute name="VALUE" x="90.932" y="50.8" size="1.27" layer="96" rot="R90"/>
+</instance>
+<instance part="R1" gate="G$1" x="95.25" y="72.39" smashed="yes" rot="R90">
+<attribute name="NAME" x="93.7514" y="68.58" size="1.27" layer="95" rot="R90"/>
+<attribute name="VALUE" x="98.552" y="68.58" size="1.27" layer="96" rot="R90"/>
+</instance>
+<instance part="GND" gate="G$1" x="10.16" y="78.74" smashed="yes">
+<attribute name="NAME" x="8.89" y="80.01" size="1.778" layer="95"/>
+<attribute name="TP_SIGNAL_NAME" x="11.43" y="77.47" size="1.778" layer="97"/>
+</instance>
+<instance part="VOUT" gate="G$1" x="12.7" y="73.66" smashed="yes">
+<attribute name="NAME" x="11.43" y="74.93" size="1.778" layer="95"/>
+<attribute name="TP_SIGNAL_NAME" x="13.97" y="72.39" size="1.778" layer="97"/>
+</instance>
+<instance part="VIN" gate="G$1" x="15.24" y="68.58" smashed="yes">
+<attribute name="NAME" x="13.97" y="69.85" size="1.778" layer="95"/>
+<attribute name="TP_SIGNAL_NAME" x="16.51" y="67.31" size="1.778" layer="97"/>
+</instance>
+<instance part="EN" gate="G$1" x="17.78" y="63.5" smashed="yes">
+<attribute name="NAME" x="16.51" y="64.77" size="1.778" layer="95"/>
+<attribute name="TP_SIGNAL_NAME" x="19.05" y="62.23" size="1.778" layer="97"/>
 </instance>
 </instances>
@@
 <net name="GND" class="0">
 <segment>
-<pinref part="SV1" gate="1" pin="1"/>
-<label x="22.86" y="43.18" size="1.27" layer="95" align="bottom-right"/>
 <pinref part="C_IN" gate="G$1" pin="1"/>
 <wire x1="30.48" y1="55.88" x2="30.48" y2="43.18" width="0.1524" layer="91"/>
-<wire x1="30.48" y1="43.18" x2="15.24" y2="43.18" width="0.1524" layer="91"/>
+<wire x1="30.48" y1="43.18" x2="10.16" y2="43.18" width="0.1524" layer="91"/>
+<wire x1="10.16" y1="43.18" x2="10.16" y2="76.2" width="0.1524" layer="91"/>
 <pinref part="U1" gate="A" pin="GND"/>
 <wire x1="73.66" y1="73.66" x2="73.66" y2="43.18" width="0.1524" layer="91"/>
@@
 <wire x1="109.22" y1="43.18" x2="87.63" y2="43.18" width="0.1524" layer="91"/>
 <junction x="87.63" y="43.18"/>
+<pinref part="GND" gate="G$1" pin="TP"/>
 </segment>
 </net>
 <net name="VOUT" class="0">
 <segment>
-<pinref part="SV1" gate="1" pin="2"/>
-<label x="22.86" y="45.72" size="1.27" layer="95" align="bottom-right"/>
 <pinref part="D1" gate="G$1" pin="C"/>
 <wire x1="77.47" y1="82.55" x2="77.47" y2="45.72" width="0.1524" layer="91"/>
-<wire x1="77.47" y1="45.72" x2="15.24" y2="45.72" width="0.1524" layer="91"/>
+<wire x1="77.47" y1="45.72" x2="12.7" y2="45.72" width="0.1524" layer="91"/>
+<wire x1="12.7" y1="45.72" x2="12.7" y2="71.12" width="0.1524" layer="91"/>
 <wire x1="77.47" y1="82.55" x2="92.71" y2="82.55" width="0.1524" layer="91"/>
 <junction x="77.47" y="82.55"/>
@@
 <wire x1="92.71" y1="82.55" x2="92.71" y2="72.39" width="0.1524" layer="91"/>
 <pinref part="C_FF" gate="G$1" pin="2"/>
-<wire x1="92.71" y1="82.55" x2="100.33" y2="82.55" width="0.1524" layer="91"/>
+<wire x1="92.71" y1="82.55" x2="95.25" y2="82.55" width="0.1524" layer="91"/>
 <junction x="92.71" y="82.55"/>
+<wire x1="95.25" y1="82.55" x2="100.33" y2="82.55" width="0.1524" layer="91"/>
 <wire x1="100.33" y1="82.55" x2="109.22" y2="82.55" width="0.1524" layer="91"/>
 <junction x="100.33" y="82.55"/>
 <pinref part="C_O" gate="G$1" pin="2"/>
 <wire x1="109.22" y1="82.55" x2="109.22" y2="66.04" width="0.1524" layer="91"/>
+<pinref part="R1" gate="G$1" pin="2"/>
+<wire x1="95.25" y1="77.47" x2="95.25" y2="82.55" width="0.1524" layer="91"/>
+<junction x="95.25" y="82.55"/>
+<pinref part="VOUT" gate="G$1" pin="TP"/>
 </segment>
 </net>
 <net name="VIN" class="0">
 <segment>
-<pinref part="SV1" gate="1" pin="3"/>
+<wire x1="15.24" y1="66.04" x2="15.24" y2="48.26" width="0.1524" layer="91"/>
 <wire x1="15.24" y1="48.26" x2="25.4" y2="48.26" width="0.1524" layer="91"/>
-<label x="22.86" y="48.26" size="1.27" layer="95" align="bottom-right"/>
 <pinref part="U1" gate="A" pin="VIN"/>
 <wire x1="38.1" y1="68.58" x2="30.48" y2="68.58" width="0.1524" layer="91"/>
@@
 <junction x="30.48" y="68.58"/>
 <pinref part="L1" gate="CD43" pin="1"/>
+<pinref part="VIN" gate="G$1" pin="TP"/>
 </segment>
 </net>
@@
 <net name="EN" class="0">
 <segment>
-<pinref part="SV1" gate="1" pin="4"/>
-<wire x1="15.24" y1="50.8" x2="20.32" y2="50.8" width="0.1524" layer="91"/>
-<label x="22.86" y="50.8" size="1.27" layer="95" align="bottom-right"/>
+<wire x1="17.78" y1="60.96" x2="17.78" y2="50.8" width="0.1524" layer="91"/>
+<wire x1="17.78" y1="50.8" x2="20.32" y2="50.8" width="0.1524" layer="91"/>
 <pinref part="U1" gate="A" pin="EN"/>
 <wire x1="38.1" y1="73.66" x2="30.48" y2="73.66" width="0.1524" layer="91"/>
@@
 <wire x1="20.32" y1="78.74" x2="25.4" y2="78.74" width="0.1524" layer="91"/>
 <junction x="25.4" y="78.74"/>
+<pinref part="EN" gate="G$1" pin="TP"/>
 </segment>
 </net>
@@
 <pinref part="C_FF" gate="G$1" pin="1"/>
 <wire x1="100.33" y1="74.93" x2="100.33" y2="62.23" width="0.1524" layer="91"/>
-<wire x1="100.33" y1="62.23" x2="87.63" y2="62.23" width="0.1524" layer="91"/>
+<wire x1="100.33" y1="62.23" x2="95.25" y2="62.23" width="0.1524" layer="91"/>
+<pinref part="R1" gate="G$1" pin="1"/>
+<wire x1="95.25" y1="62.23" x2="87.63" y2="62.23" width="0.1524" layer="91"/>
+<wire x1="95.25" y1="67.31" x2="95.25" y2="62.23" width="0.1524" layer="91"/>
+<junction x="95.25" y="62.23"/>
 </segment>
 </net>
@@
 for full support of SPICE simulation.
 </note>
-<note version="9.0" severity="warning">
-Since Version 9.0, EAGLE supports the align property for labels.
-Labels in schematic will not be understood with this version. Update EAGLE to the latest version
-for full support of labels.
-</note>
 </compatibility>

Commit message: update to v1.2
Parts:
- removed EN, GND, VIN, VOUT: TPB1,27, testpad:TPB1,27
- added J2: (no value), SparkFun-Connectors:CONN_041X04_NO_SILK
- D1: value SS54 -> SS14
- R1: value Xk -> xxxk
- R2: value 1k -> 100k
- U1: value TPS61040DBVR -> TPS61040
- VR1: value 10k -> 1M
Connections:
- net EN: now also J2.4; no longer EN.TP
- net GND: now also J2.1; no longer GND.TP
- net VIN: now also J2.3; no longer VIN.TP
- net VOUT: now also J2.2; no longer VOUT.TP
Other:
- moved on the sheet: C_FF, C_IN, C_O, D1, EN_J, L1, R1, R2, U1, VR1
